File: PCB/PlaiKeyboard.kicad_pcb (KiCad board)
At the start: 2 copper layers, 374.4 x 139.2 mm, 172 parts, among them SW1 SW_Push_45deg, SW10 SW_Push_45deg, SW11 SW_Push_45deg, SW12 SW_Push_45deg, SW13 SW_Push_45deg, SW14 SW_Push_45deg, SW15 RotaryEncoder_Switch, SW16 SW_Push_45deg, SW17 SW_Push_45deg, SW18 SW_Push_45deg, SW19 SW_Push_45deg, SW2 SW_Push_45deg, SW20 SW_Push_45deg, SW21 SW_Push_45deg, SW22 SW_Push_45deg, SW23 SW_Push_45deg, SW24 SW_Push_45deg, SW25 SW_Push_45deg, SW26 SW_Push_45deg, SW27 SW_Push_45deg, SW28 SW_Push_45deg, SW29 SW_Push_45deg, SW3 SW_Push_45deg, SW30 SW_Push_45deg, SW31 SW_Push_45deg, SW32 SW_Push_45deg, SW33 SW_Push_45deg, SW34 SW_Push_45deg, SW35 SW_Push_45deg, SW36 SW_Push_45deg, SW37 SW_Push_45deg, SW38 SW_Push_45deg, SW39 SW_Push_45deg, SW4 SW_Push_45deg, SW40 SW_Push_45deg, SW41 SW_Push_45deg, SW42 SW_Push_45deg, SW43 SW_Push_45deg, SW44 SW_Push_45deg, SW45 SW_Push_45deg, SW46 SW_Push_45deg, SW47 SW_Push_45deg, SW48 SW_Push_45deg, SW49 SW_Push_45deg, SW5 SW_Push_45deg, SW50 SW_Push_45deg, SW51 SW_Push_45deg, SW52 SW_Push_45deg, SW53 SW_Push_45deg, SW54 SW_Push_45deg, SW55 SW_Push_45deg, SW56 SW_Push_45deg, SW57 SW_Push_45deg, SW58 SW_Push_45deg, SW59 SW_Push_45deg, SW6 SW_Push_45deg, SW60 SW_Push_45deg, SW61 SW_Push_45deg, SW62 SW_Push_45deg, SW63 SW_Push_45deg, SW64 SW_Push_45deg, SW65 SW_Push_45deg, SW66 SW_Push_45deg, SW67 SW_Push_45deg, SW68 SW_Push_45deg, SW69 SW_Push_45deg, SW7 SW_Push_45deg, SW70 SW_Push_45deg, SW71 SW_Push_45deg, SW72 SW_Push_45deg, SW73 SW_Push_45deg, SW74 SW_Push_45deg, SW75 SW_Push_45deg, SW76 SW_Push_45deg, SW77 SW_Push_45deg, SW78 SW_Push_45deg, SW79 SW_Push_45deg, SW8 SW_Push_45deg, SW80 SW_Push_45deg, SW81 SW_Push_45deg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

Commit message: Commit
Parts:
- removed C3: 100nF, Capacitor_THT:C_Rect_L11.5mm_W5.2mm_P10.00mm_MKT
- removed SW1: SW_Push_45deg, Button_Switch_Keyboard:SW_Cherry_MX_1.00u_PCB
- removed U2: 74HC595, Package_DIP:DIP-16_W7.62mm_LongPads
- added SW84: SW_Push_45deg, Button_Switch_Keyboard:SW_Cherry_MX_1.00u_PCB, F.Cu at (309.6, 128.6)
- C1: value 100nF -> 10µF; footprint Capacitor_THT:C_Rect_L11.5mm_W5.2mm_P10.00mm_MKT -> Capacitor_THT:C_Disc_D4.7mm_W2.5mm_P5.00mm
- C2: value 10µF -> 100nF; footprint Capacitor_THT:C_Disc_D4.7mm_W2.5mm_P5.00mm -> Capacitor_THT:C_Rect_L11.5mm_W5.2mm_P10.00mm_MKT
- D61: moved to F.Cu
- SW15: value RotaryEncoder_Switch -> SW_Push_45deg; footprint Rotary_Encoder:RotaryEncoder_Alps_EC11E-Switch_Vertical_H20mm -> Button_Switch_Keyboard:SW_Cherry_MX_1.25u_PCB
- SW22, SW8: footprint Button_Switch_Keyboard:SW_Cherry_MX_1.00u_PCB -> Button_Switch_Keyboard:SW_Cherry_MX_1.25u_PCB
- SW25: footprint Button_Switch_Keyboard:SW_Cherry_MX_1.00u_PCB -> Button_Switch_Keyboard:SW_Cherry_MX_2.00u_PCB
- SW29: footprint Button_Switch_Keyboard:SW_Cherry_MX_2.00u_PCB -> Button_Switch_Keyboard:SW_Cherry_MX_6.25u_PCB
- SW31, SW44: footprint Button_Switch_Keyboard:SW_Cherry_MX_1.50u_PCB -> Button_Switch_Keyboard:SW_Cherry_MX_1.00u_PCB
- SW39, SW47: footprint Button_Switch_Keyboard:SW_Cherry_MX_1.00u_PCB -> Button_Switch_Keyboard:SW_Cherry_MX_1.50u_PCB
- SW46, SW71: footprint Button_Switch_Keyboard:SW_Cherry_MX_1.75u_PCB -> Button_Switch_Keyboard:SW_Cherry_MX_1.00u_PCB
- SW58, SW60: footprint Button_Switch_Keyboard:SW_Cherry_MX_2.25u_PCB -> Button_Switch_Keyboard:SW_Cherry_MX_1.00u_PCB
- SW61, SW70: footprint Button_Switch_Keyboard:SW_Cherry_MX_1.00u_PCB -> Button_Switch_Keyboard:SW_Cherry_MX_1.75u_PCB
- SW62: footprint Button_Switch_Keyboard:SW_Cherry_MX_1.00u_PCB -> Button_Switch_Keyboard:SW_Cherry_MX_2.25u_PCB
- SW74, SW75: footprint Button_Switch_Keyboard:SW_Cherry_MX_1.25u_PCB -> Button_Switch_Keyboard:SW_Cherry_MX_1.00u_PCB
- SW76: footprint Button_Switch_Keyboard:SW_Cherry_MX_1.25u_PCB -> Button_Switch_Keyboard:SW_Cherry_MX_2.25u_PCB
- SW77: footprint Button_Switch_Keyboard:SW_Cherry_MX_6.25u_PCB -> Button_Switch_Keyboard:SW_Cherry_MX_1.00u_PCB
- SW78: value SW_Push_45deg -> RotaryEncoder_Switch; footprint Button_Switch_Keyboard:SW_Cherry_MX_1.00u_PCB -> Rotary_Encoder:RotaryEncoder_Alps_EC11E-Switch_Vertical_H20mm
- moved SW15 354.1 mm to (64.3, 138.1)
- moved SW83 336.7 mm to (81.0, 119.1)
- moved D82 336.5 mm to (88.0, 127.3)
- moved D14 328.2 mm to (71.2, 146.3)
- moved SW45 307.0 mm to (114.3, 61.9)
- moved D44 306.8 mm to (121.5, 70.3)
- moved SW30 303.0 mm to (119.1, 38.1)
- moved D29 303.0 mm to (126.1, 46.3)
- moved SW82 293.4 mm to (109.5, 100.0)
- moved D81 293.3 mm to (116.6, 108.3)
- moved SW59 272.7 mm to (152.4, 61.9)
- moved D58 272.4 mm to (159.6, 70.3)
- moved SW14 270.7 mm to (119.1, 119.1)
- moved D13 247.2 mm to (126.2, 127.3)
- moved D38 236.2 mm to (49.6, 88.3)
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Connections:
- C1 pad 1: +3V3 -> GND
- C1 pad 2: GND -> /VBAT_SW
- C2 pad 1: GND -> +3V3
- C2 pad 2: /VBAT_SW -> GND
- D10 pad 1: ROW0 -> ROW2
- D11 pad 1: ROW0 -> ROW3
- D12 pad 1: ROW0 -> ROW4
- D13 pad 1: ROW0 -> ROW5
- D14 pad 1: ROW0 -> ROW6
- D15 pad 1: ROW1 -> ROW0
- D17 pad 1: ROW1 -> ROW2
- D18 pad 1: ROW1 -> ROW3
- D19 pad 1: ROW1 -> ROW4
- D2 pad 1: ROW0 -> ROW1
- D20 pad 1: ROW1 -> ROW5
- D21 pad 1: ROW1 -> ROW6
- D22 pad 1: ROW1 -> ROW0
- D24 pad 1: ROW1 -> ROW2
- D25 pad 1: ROW1 -> ROW3
- D26 pad 1: ROW1 -> ROW4
- D27 pad 1: ROW1 -> ROW5
- D28 pad 1: ROW1 -> ROW6
- D29 pad 1: ROW1 -> ROW0
- D3 pad 1: ROW0 -> ROW2
- D30 pad 1: ROW2 -> ROW1
- D32 pad 1: ROW2 -> ROW3
- D33 pad 1: ROW2 -> ROW4
- D34 pad 1: ROW2 -> ROW5
- D35 pad 1: ROW2 -> ROW6
- D36 pad 1: ROW2 -> ROW0
- D37 pad 1: ROW2 -> ROW1
- D39 pad 1: ROW2 -> ROW3
- D4 pad 1: ROW0 -> ROW3
- D40 pad 1: ROW2 -> ROW4
- D41 pad 1: ROW2 -> ROW5
- D42 pad 1: ROW2 -> ROW6
- D43 pad 1: ROW2 -> ROW0
- D44 pad 1: ROW2 -> ROW1
- D45 pad 1: ROW3 -> ROW2
- D47 pad 1: ROW3 -> ROW4
- D48 pad 1: ROW3 -> ROW5
- D49 pad 1: ROW3 -> ROW6
- D5 pad 1: ROW0 -> ROW4
- D50 pad 1: ROW3 -> ROW0
- D51 pad 1: ROW3 -> ROW1
- D52 pad 1: ROW3 -> ROW2
- D54 pad 1: ROW3 -> ROW4
- D55 pad 1: ROW3 -> ROW5
- D56 pad 1: ROW3 -> ROW6
- D57 pad 1: ROW3 -> ROW0
- D58 pad 1: ROW3 -> ROW1
- D59 pad 1: ROW4 -> ROW2
- D6 pad 1: ROW0 -> ROW5
- D60 pad 1: ROW4 -> ROW3
- D62 pad 1: ROW4 -> ROW5
- D63 pad 1: ROW4 -> ROW6
- D64 pad 1: ROW4 -> ROW0
- D65 pad 1: ROW4 -> ROW1
- D66 pad 1: ROW4 -> ROW2
- D67 pad 1: ROW4 -> ROW3
- D69 pad 1: ROW4 -> ROW5
- D7 pad 1: ROW0 -> ROW6
- D70 pad 1: ROW4 -> ROW6
- D71 pad 1: ROW4 -> ROW0
- D72 pad 1: ROW4 -> ROW1
- D73 pad 1: ROW5 -> ROW2
- D74 pad 1: ROW5 -> ROW3
- D75 pad 1: ROW5 -> ROW4
- D77 pad 1: ROW5 -> ROW6
- D78 pad 1: ROW5 -> ROW0
- D79 pad 1: ROW5 -> ROW1
- D80 pad 1: ROW5 -> ROW2
- D81 pad 1: ROW5 -> ROW3
- D82 pad 1: ROW5 -> ROW4
- D83 pad 1: ROW0 -> ROW5
- D9 pad 1: ROW0 -> ROW1
- SW10 pad 1: COL9 -> COL1
- SW10 pad 2: Net-(D10-A) -> Net-(D9-A)
- SW11 pad 1: COL10 -> COL1
- SW11 pad 2: Net-(D11-A) -> Net-(D10-A)
- SW12 pad 1: COL11 -> COL1
- SW12 pad 2: Net-(D12-A) -> Net-(D11-A)
- SW13 pad 1: COL12 -> COL1
- SW13 pad 2: Net-(D13-A) -> Net-(D12-A)
- SW14 pad 1: COL13 -> COL1
- SW14 pad 2: Net-(D14-A) -> Net-(D13-A)
- SW16 pad 1: COL0 -> COL2
- SW17 pad 1: COL1 -> COL2
- SW19 pad 1: COL3 -> COL2
- SW2 pad 1: COL1 -> COL0
- SW2 pad 2: Net-(D2-A) -> Net-(D1-A)
- SW20 pad 1: COL4 -> COL2
- SW21 pad 1: COL5 -> COL2
- SW22 pad 1: COL6 -> COL2
- SW23 pad 1: COL7 -> COL3
- SW24 pad 1: COL8 -> COL3
- SW25 pad 1: COL9 -> COL3
- SW26 pad 1: COL10 -> COL3
- SW27 pad 1: COL11 -> COL3
- SW28 pad 1: COL12 -> COL3
- SW29 pad 1: COL13 -> COL3
- SW3 pad 1: COL2 -> COL0
- SW3 pad 2: Net-(D3-A) -> Net-(D2-A)
- SW30 pad 1: COL14 -> COL4
- SW31 pad 1: COL0 -> COL4
- SW32 pad 1: COL1 -> COL4
- SW33 pad 1: COL2 -> COL4
- SW34 pad 1: COL3 -> COL4
- SW36 pad 1: COL5 -> COL4
- SW37 pad 1: COL6 -> COL5
- SW38 pad 1: COL7 -> COL5
- SW39 pad 1: COL8 -> COL5
- SW4 pad 1: COL3 -> COL0
- SW4 pad 2: Net-(D4-A) -> Net-(D3-A)
- SW40 pad 1: COL9 -> COL5
- SW41 pad 1: COL10 -> COL5
- SW42 pad 1: COL11 -> COL5
- SW43 pad 1: COL12 -> COL5
- SW44 pad 1: COL13 -> COL6
- SW45 pad 1: COL14 -> COL6
- SW46 pad 1: COL0 -> COL6
- SW47 pad 1: COL1 -> COL6
- SW48 pad 1: COL2 -> COL6
- SW49 pad 1: COL3 -> COL6
- SW5 pad 1: COL4 -> COL0
- SW5 pad 2: Net-(D5-A) -> Net-(D4-A)
- SW50 pad 1: COL4 -> COL6
- SW51 pad 1: COL5 -> COL7
- SW52 pad 1: COL6 -> COL7
- SW54 pad 1: COL8 -> COL7
- SW55 pad 1: COL9 -> COL7
- SW56 pad 1: COL10 -> COL7
- SW57 pad 1: COL11 -> COL7
- SW58 pad 1: COL12 -> COL8
- SW59 pad 1: COL13 -> COL8
- SW6 pad 1: COL5 -> COL0
- SW6 pad 2: Net-(D6-A) -> Net-(D5-A)
- SW60 pad 1: COL0 -> COL8
- SW61 pad 1: COL1 -> COL8
- SW62 pad 1: COL2 -> COL8
- SW63 pad 1: COL3 -> COL8
- SW64 pad 1: COL4 -> COL8
- SW65 pad 1: COL5 -> COL9
- SW66 pad 1: COL6 -> COL9
- SW67 pad 1: COL7 -> COL9
- SW68 pad 1: COL8 -> COL9
- SW7 pad 1: COL6 -> COL0
- SW7 pad 2: Net-(D7-A) -> Net-(D6-A)
- SW70 pad 1: COL10 -> COL9
- SW71 pad 1: COL11 -> COL9
- SW72 pad 1: COL12 -> COL10
- SW73 pad 1: COL13 -> COL10
- SW74 pad 1: COL0 -> COL10
- SW75 pad 1: COL1 -> COL10
- SW76 pad 1: COL2 -> COL10
- SW77 pad 1: COL3 -> COL10
- SW79 pad 1: COL5 -> COL11
- SW8 pad 1: COL7 -> COL0
- SW8 pad 2: Net-(D8-A) -> Net-(D7-A)
- SW80 pad 1: COL6 -> COL11
- SW81 pad 1: COL7 -> COL11
- SW82 pad 1: COL8 -> COL11
- SW83 pad 1: COL9 -> COL11
- SW9 pad 1: COL8 -> COL1
- SW9 pad 2: Net-(D9-A) -> Net-(D8-A)
- U1 pad 10: ROW2 -> ROW5
- U1 pad 11: ROW3 -> ROW6
- U1 pad 12: ROW4 -> COL0
- U1 pad 17: COL2 -> COL4
- U1 pad 18: COL3 -> COL5
- U1 pad 19: COL4 -> COL6
- U1 pad 20: COL5 -> COL7
- U1 pad 21: COL6 -> COL8
- U1 pad 22: COL7 -> COL9
- U1 pad 23: COL8 -> COL10
- U1 pad 24: COL9 -> COL11
- U1 pad 25: ROW5 -> COL1
- U1 pad 26: COL0 -> COL2
- U1 pad 27: COL1 -> COL3
- U1 pad 5: SR_CLOCK -> ROW0
- U1 pad 6: SR_DATA -> ROW1
- U1 pad 7: SR_LATCH -> ROW2
- U1 pad 8: ROW0 -> ROW3
- U1 pad 9: ROW1 -> ROW4
Routing:
- net ROW6: track 0.00 -> 439.3 mm, vias 0 -> 2
- net COL10: track 230.7 -> 544.7 mm
- net COL6: track 356.0 -> 632.9 mm, vias 0 -> 1
- net COL11: track 209.4 -> 473.9 mm, vias 0 -> 7
- net ROW3: track 586.6 -> 343.8 mm, vias 0 -> 2
- net COL3: track 433.8 -> 667.6 mm, vias 0 -> 2
- net COL8: track 451.7 -> 680.7 mm
- net COL5: track 381.5 -> 600.8 mm, vias 2 -> 0
- net COL7: track 344.7 -> 546.4 mm, vias 2 -> 6
- net COL12: track 185.7 -> 0.00 mm, vias 1 -> 0
- net COL13: track 178.2 -> 0.00 mm, vias 1 -> 0
- net COL9: track 413.5 -> 580.7 mm, vias 1 -> 2
- net COL4: track 393.1 -> 493.4 mm, vias 2 -> 6
- net ROW4: track 447.7 -> 347.7 mm, vias 0 -> 3
- net ROW5: track 408.2 -> 318.9 mm
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Other:
- board size 374.4 x 139.2 mm -> 370 x 140 mm
- board text added: "Plaikeyboard"
- board text added: "What you doing here?"
