File: PCB/_restore_backup_2026-08-09T21-39-08-163/PlaiKeyboard.kicad_pcb (KiCad board)
At the start: 2 copper layers, 374.4 x 139.2 mm, 172 parts, among them SW1 SW_Push_45deg, SW10 SW_Push_45deg, SW11 SW_Push_45deg, SW12 SW_Push_45deg, SW13 SW_Push_45deg, SW14 SW_Push_45deg, SW15 RotaryEncoder_Switch, SW16 SW_Push_45deg, SW17 SW_Push_45deg, SW18 SW_Push_45deg, SW19 SW_Push_45deg, SW2 SW_Push_45deg, SW20 SW_Push_45deg, SW21 SW_Push_45deg, SW22 SW_Push_45deg, SW23 SW_Push_45deg, SW24 SW_Push_45deg, SW25 SW_Push_45deg, SW26 SW_Push_45deg, SW27 SW_Push_45deg, SW28 SW_Push_45deg, SW29 SW_Push_45deg, SW3 SW_Push_45deg, SW30 SW_Push_45deg, SW31 SW_Push_45deg, SW32 SW_Push_45deg, SW33 SW_Push_45deg, SW34 SW_Push_45deg, SW35 SW_Push_45deg, SW36 SW_Push_45deg, SW37 SW_Push_45deg, SW38 SW_Push_45deg, SW39 SW_Push_45deg, SW4 SW_Push_45deg, SW40 SW_Push_45deg, SW41 SW_Push_45deg, SW42 SW_Push_45deg, SW43 SW_Push_45deg, SW44 SW_Push_45deg, SW45 SW_Push_45deg, SW46 SW_Push_45deg, SW47 SW_Push_45deg, SW48 SW_Push_45deg, SW49 SW_Push_45deg, SW5 SW_Push_45deg, SW50 SW_Push_45deg, SW51 SW_Push_45deg, SW52 SW_Push_45deg, SW53 SW_Push_45deg, SW54 SW_Push_45deg, SW55 SW_Push_45deg, SW56 SW_Push_45deg, SW57 SW_Push_45deg, SW58 SW_Push_45deg, SW59 SW_Push_45deg, SW6 SW_Push_45deg, SW60 SW_Push_45deg, SW61 SW_Push_45deg, SW62 SW_Push_45deg, SW63 SW_Push_45deg, SW64 SW_Push_45deg, SW65 SW_Push_45deg, SW66 SW_Push_45deg, SW67 SW_Push_45deg, SW68 SW_Push_45deg, SW69 SW_Push_45deg, SW7 SW_Push_45deg, SW70 SW_Push_45deg, SW71 SW_Push_45deg, SW72 SW_Push_45deg, SW73 SW_Push_45deg, SW74 SW_Push_45deg, SW75 SW_Push_45deg, SW76 SW_Push_45deg, SW77 SW_Push_45deg, SW78 SW_Push_45deg, SW79 SW_Push_45deg, SW8 SW_Push_45deg, SW80 SW_Push_45deg, SW81 SW_Push_45deg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

Commit message: ACTUALLY FINISHED WITH THE PCB
Parts:
- removed C1, C3: 100nF, Capacitor_THT:C_Rect_L11.5mm_W5.2mm_P10.00mm_MKT
- removed C2: 10µF, Capacitor_THT:C_Disc_D4.7mm_W2.5mm_P5.00mm
- removed J_BAT1: GND, Connector_JST:JST_PH_S2B-PH-K_1x02_P2.00mm_Horizontal
- removed U1: SuperMini nRF52840, PCM_marbastlib-xp-promicroish:SuperMini_nRF52840_AH_USBup
- removed U2: 74HC595, Package_DIP:DIP-16_W7.62mm_LongPads
- added A1: RaspberryPi_Pico, Module:RaspberryPi_Pico_Common_Unspecified, F.Cu at (456.5, 77.5)
Routing:
- net ROW3: track 586.6 -> 160.9 mm, vias 0 -> 2
- net ROW4: track 447.7 -> 101.4 mm, vias 0 -> 3
- net ROW2: track 343.1 -> 0.00 mm
- net ROW1: track 331.0 -> 0.00 mm
- net ROW5: track 408.2 -> 111.6 mm
- net ROW0: track 323.9 -> 50.5 mm, vias 0 -> 1
- net COL8: track 451.7 -> 190.7 mm, vias 1 -> 2
- net COL9: track 413.5 -> 167.9 mm
- net COL0: track 517.8 -> 349.1 mm
- net COL1: track 475.2 -> 323.1 mm
- net GND: track 147.6 -> 0.00 mm
- net COL5: track 381.5 -> 243.6 mm, vias 2 -> 1
- net COL7: track 344.7 -> 208.2 mm
- net COL3: track 433.8 -> 301.1 mm
- net COL4: track 393.1 -> 261.7 mm
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Other:
- board size 374.4 x 139.2 mm -> 374.5 x 139 mm
