File: PCB/_restore_backup_2026-08-11T06-42-38-122/PlaiKeyboard.kicad_pcb (KiCad board)
At the start: 2 copper layers, 374.4 x 139.2 mm, 172 parts, among them SW1 SW_Push_45deg, SW10 SW_Push_45deg, SW11 SW_Push_45deg, SW12 SW_Push_45deg, SW13 SW_Push_45deg, SW14 SW_Push_45deg, SW15 RotaryEncoder_Switch, SW16 SW_Push_45deg, SW17 SW_Push_45deg, SW18 SW_Push_45deg, SW19 SW_Push_45deg, SW2 SW_Push_45deg, SW20 SW_Push_45deg, SW21 SW_Push_45deg, SW22 SW_Push_45deg, SW23 SW_Push_45deg, SW24 SW_Push_45deg, SW25 SW_Push_45deg, SW26 SW_Push_45deg, SW27 SW_Push_45deg, SW28 SW_Push_45deg, SW29 SW_Push_45deg, SW3 SW_Push_45deg, SW30 SW_Push_45deg, SW31 SW_Push_45deg, SW32 SW_Push_45deg, SW33 SW_Push_45deg, SW34 SW_Push_45deg, SW35 SW_Push_45deg, SW36 SW_Push_45deg, SW37 SW_Push_45deg, SW38 SW_Push_45deg, SW39 SW_Push_45deg, SW4 SW_Push_45deg, SW40 SW_Push_45deg, SW41 SW_Push_45deg, SW42 SW_Push_45deg, SW43 SW_Push_45deg, SW44 SW_Push_45deg, SW45 SW_Push_45deg, SW46 SW_Push_45deg, SW47 SW_Push_45deg, SW48 SW_Push_45deg, SW49 SW_Push_45deg, SW5 SW_Push_45deg, SW50 SW_Push_45deg, SW51 SW_Push_45deg, SW52 SW_Push_45deg, SW53 SW_Push_45deg, SW54 SW_Push_45deg, SW55 SW_Push_45deg, SW56 SW_Push_45deg, SW57 SW_Push_45deg, SW58 SW_Push_45deg, SW59 SW_Push_45deg, SW6 SW_Push_45deg, SW60 SW_Push_45deg, SW61 SW_Push_45deg, SW62 SW_Push_45deg, SW63 SW_Push_45deg, SW64 SW_Push_45deg, SW65 SW_Push_45deg, SW66 SW_Push_45deg, SW67 SW_Push_45deg, SW68 SW_Push_45deg, SW69 SW_Push_45deg, SW7 SW_Push_45deg, SW70 SW_Push_45deg, SW71 SW_Push_45deg, SW72 SW_Push_45deg, SW73 SW_Push_45deg, SW74 SW_Push_45deg, SW75 SW_Push_45deg, SW76 SW_Push_45deg, SW77 SW_Push_45deg, SW78 SW_Push_45deg, SW79 SW_Push_45deg, SW8 SW_Push_45deg, SW80 SW_Push_45deg, SW81 SW_Push_45deg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

Commit message: ACTUALLY FINISHED WITH THE PCB
Routing:
- net COL8: track 451.7 -> 209.3 mm, vias 1 -> 2
- net ROW3: track 586.6 -> 355.4 mm, vias 0 -> 2
- net COL4: track 393.1 -> 191.2 mm
- net COL9: track 413.5 -> 212.3 mm
- net COL3: track 433.8 -> 624.3 mm
- net COL5: track 381.5 -> 193.1 mm, vias 2 -> 1
- net COL6: track 356.0 -> 196.4 mm, vias 0 -> 1
- net GND: track 147.6 -> 0.00 mm
- net COL7: track 344.7 -> 209.5 mm
- net COL10: track 230.7 -> 96.7 mm
- net COL11: track 209.4 -> 99.7 mm
- net COL13: track 178.2 -> 97.5 mm, vias 1 -> 2
- net ROW4: track 447.7 -> 368.2 mm, vias 0 -> 3
- net +3V3: track 63.6 -> 0.00 mm
- net COL12: track 185.7 -> 134.9 mm, vias 1 -> 2
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Other:
- board size 374.4 x 139.2 mm -> 374.5 x 139 mm
